Commit message: fixed simulator launch scripts

File: src/tardigrade/urdf/tardigrade_base.urdf.xacro (robot description, xacro)
@@ -17,5 +17,5 @@
      limitations under the License.
 -->
-<robot xmlns:xacro="http://www.ros.org/wiki/xacro">
+<robot xmlns:xacro="http://www.ros.org/wiki/xacro" name='tardigrade'>
   <!--
       The RexROV meshes and hydrodynamic parameters are based on the parameters and dimensions
@@ -28,6 +28,6 @@
   <!-- includes -->
   <xacro:include filename="$(find tardigrade)/urdf/common.urdf.xacro"/>
-  <xacro:include filename="$(find tardigrade)/urdf/sensor_snippets.xacro"/>
-  <xacro:include filename="$(find tardigrade)/urdf/snippets.xacro"/>
+  <xacro:include filename="$(find uuv_sensor_ros_plugins)/urdf/sensor_snippets.xacro"/>
+  <xacro:include filename="$(find uuv_gazebo_ros_plugins)/urdf/snippets.xacro"/>
   <!-- Parameters -->
   <xacro:property name="namespace" value="tardigrade"/>
@@ -36,5 +36,5 @@
   <!-- Mass, see p.28 in Berg2012 -->
   <xacro:property name="mass" value="1862.87"/>
-  <xacro:macro name="rexrov_base" params="namespace *gazebo inertial_reference_frame">
+  <xacro:macro name="tardigrade_base" params="namespace *gazebo inertial_reference_frame">
     <!-- base_link according to ROS conventions: x forward, z up -->
     <link name="${namespace}/base_link">
@@ -47,5 +47,5 @@
         <origin xyz="0 0 0" rpy="0 0 0"/>
         <geometry>
-          <mesh filename="${visual_mesh_file}" scale="1 1 1"/>
+          <mesh filename="${visual_mesh_file}" scale="0.005 0.005 0.005"/>
         </geometry>
       </visual>
@@ -83,3 +83,6 @@
     <xacro:include filename="$(find tardigrade)/urdf/tardigrade_sensors.xacro"/>
   </xacro:macro>
+  <xacro:tardigrade_base namespace="${namespace}" inertial_reference_frame="world">
+    <gazebo/>
+  </xacro:tardigrade_base>
 </robot>
