Commit message: added gate approach and update xacros

File: src/tardigrade/urdf/tardigrade_actuators.xacro (robot description, xacro)
@@ -32,26 +32,26 @@
   </xacro:macro>
   <xacro:thruster_macro namespace="${namespace}" thruster_id="0">
-    <origin xyz="0.259 0.173026 0.50891" rpy="${0*d2r} ${0*d2r} ${-45*d2r}"/>
+    <origin xyz="-0.890895 0.334385 0.528822" rpy="${0*d2r} ${-74.53*d2r} ${-53.21*d2r}"/>
   </xacro:thruster_macro>
   <xacro:thruster_macro namespace="${namespace}" thruster_id="1">
-    <origin xyz="0.259 -0.173026 0.50891" rpy="${0*d2r} ${0*d2r} ${45*d2r}"/>
+    <origin xyz="-0.890895 -0.334385 0.528822" rpy="${0*d2r} ${-74.53*d2r} ${53.21*d2r}"/>
   </xacro:thruster_macro>
   <xacro:thruster_macro namespace="${namespace}" thruster_id="2">
-    <origin xyz="-0.259 0.173026 0.50891" rpy="${0*d2r} ${0*d2r} ${-135*d2r}"/>
+    <origin xyz="0.890895 0.334385 0.528822" rpy="${0*d2r} ${-105.47*d2r} ${53.21*d2r}"/>
   </xacro:thruster_macro>
   <xacro:thruster_macro namespace="${namespace}" thruster_id="3">
-    <origin xyz="-0.259 -0.173026 0.50891" rpy="${0*d2r} ${0*d2r} ${135*d2r}"/>
+    <origin xyz="0.890895 -0.334385 0.528822" rpy="${0*d2r} ${-105.47*d2r} ${-53.21*d2r}"/>
   </xacro:thruster_macro>
   <xacro:thruster_macro namespace="${namespace}" thruster_id="4">
-    <origin xyz="0.092485 0.189603 -0.095324" rpy="${-90*d2r} ${0*d2r} ${0*d2r}"/>
+    <origin xyz="-0.412125 0.505415 0.129" rpy="${0*d2r} ${0*d2r} ${45*d2r}"/>
   </xacro:thruster_macro>
   <xacro:thruster_macro namespace="${namespace}" thruster_id="5">
-    <origin xyz="0.092485 -0.189603 -0.095324" rpy="${-90*d2r} ${0*d2r} ${0*d2r}"/>
+    <origin xyz="-0.412125 -0.505415 0.129" rpy="${0*d2r} ${0*d2r} ${-45*d2r}"/>
   </xacro:thruster_macro>
   <xacro:thruster_macro namespace="${namespace}" thruster_id="6">
-    <origin xyz="-0.092485 0.189603 -0.095324" rpy="${-90*d2r} ${0*d2r} ${0*d2r}"/>
+    <origin xyz="0.412125 0.505415 0.129" rpy="${0*d2r} ${0*d2r} ${135*d2r}"/>
   </xacro:thruster_macro>
   <xacro:thruster_macro namespace="${namespace}" thruster_id="7">
-    <origin xyz="-0.092485 -0.189603 -0.095324" rpy="${-90*d2r} ${0*d2r} ${0*d2r}"/>
+    <origin xyz="0.412125 -0.505415 0.129" rpy="${0*d2r} ${0*d2r} ${-135*d2r}"/>
   </xacro:thruster_macro>
 </robot>

File: src/tardigrade/urdf/tardigrade_base.xacro (robot description, xacro)
@@ -17,5 +17,5 @@
      limitations under the License.
 -->
-<robot xmlns:xacro="http://www.ros.org/wiki/xacro" name='tardigrade'>
+<robot xmlns:xacro="http://www.ros.org/wiki/xacro">
   <!--
       The RexROV meshes and hydrodynamic parameters are based on the parameters and dimensions
@@ -32,5 +32,5 @@
   <!-- Parameters -->
   <xacro:property name="namespace" value="tardigrade"/>
-  <xacro:property name="visual_mesh_file" value="file://$(find tardigrade)/meshes/tardigrade_no_props.STL"/>
+  <xacro:property name="visual_mesh_file" value="file://$(find tardigrade)/meshes/RexROV_no_props.dae"/>
   <xacro:property name="prop_mesh_file" value="file://$(find tardigrade)/meshes/prop.dae"/>
   <!-- Mass, see p.28 in Berg2012 -->
@@ -47,5 +47,5 @@
         <origin xyz="0 0 0" rpy="0 0 0"/>
         <geometry>
-          <mesh filename="${visual_mesh_file}" scale="0.005 0.005 0.005"/>
+          <mesh filename="${visual_mesh_file}" scale="1 1 1"/>
         </geometry>
       </visual>
