Commit message: fixed plankton physics

File: src/tardigrade/robots/tardigrade_default.xacro (robot description, xacro)
@@ -17,13 +17,13 @@
      limitations under the License.
 -->
-<robot name="rexrov" xmlns:xacro="http://www.ros.org/wiki/xacro" >
+<robot name="tardigrade" xmlns:xacro="http://www.ros.org/wiki/xacro" >
   <xacro:arg name="debug" default="0"/>
-  <xacro:arg name="namespace" default="rexrov"/>
+  <xacro:arg name="namespace" default="tardigrade"/>
   <xacro:arg name="inertial_reference_frame" default="world"/>
   <!-- Include the ROV macro file -->
-  <xacro:include filename="$(find uuv_descriptions)/urdf/rexrov_base.xacro"/>
-  <xacro:include filename="$(find uuv_descriptions)/urdf/rexrov.gazebo.xacro"/>
+  <xacro:include filename="$(find tardigrade)/urdf/tardigrade_base.xacro"/>
+  <xacro:include filename="$(find tardigrade)/urdf/tardigrade.gazebo.xacro"/>
   <!-- Create the rexrov -->
-  <xacro:rexrov_base
+  <xacro:tardigrade_base
     namespace="$(arg namespace)"
     inertial_reference_frame="$(arg inertial_reference_frame)">
@@ -36,8 +36,8 @@
         <debug>$(arg debug)</debug>
         <!-- Adding the hydrodynamic and hydrostatic parameters for the vehicle-->
-        <xacro:rexrov_hydro_model namespace="$(arg namespace)"/>
+        <xacro:tardigrade_hydro_model namespace="$(arg namespace)"/>
       </plugin>
     </gazebo>
-  </xacro:rexrov_base>
+  </xacro:tardigrade_base>
   <!-- Joint state publisher plugin -->
   <xacro:default_joint_state_publisher namespace="$(arg namespace)" update_rate="50"/>

File: src/tardigrade/urdf/tardigrade.gazebo.xacro (robot description, xacro)
@@ -26,5 +26,5 @@
     <!-- Volume, see p.31 in Berg2012 -->
     <xacro:property name="volume" value="1.83826"/>
-    <xacro:macro name="rexrov_hydro_model" params="namespace">
+    <xacro:macro name="tardigrade_hydro_model" params="namespace">
         <link name="${namespace}/base_link">
             <neutrally_buoyant>0</neutrally_buoyant>
